File: CalibrationBoard.sch (EAGLE design)
At the start: 56 parts, among them Q1 N-HEXFET-2D_SOT232-, U1 MAX6225ACSA+, U2 MAX6250ACSA+, U3 MAX6126AASA50+

Commit message: Updates to CAD layout
moved TH to top side, SMDs are on bottom side
Parts:
- removed BAT2: (no value), SparkFun-Connectors:BC9VPC
- removed J10, J11: (no value), SparkFun-Connectors:BANANA_CONN
- removed JP1, JP2: (no value), pinhead:PINHD-1X2
- removed S1: (no value), adafruit:EG1218S
- removed TM1, TM2: 10k, adafruit:TRIMPOTTC33X
- added D1: (no value), diode:DIODE-2AC|CATO220V
- added F1: 12A, fuse:FUSELITTLEFUSE
- added F2: 1.1A, adafruit:PTCFUSE-1812
- added KK2: SK104-PAD, heatsink:SK104-PAD
- added LOGO1: OSHW-LOGOL, SparkFun-Aesthetics:OSHW-LOGOL
- added PAD1, PAD2, PAD3, PAD4, PAD5, PAD6: (no value), wirepad:3,81/1,4
- added S3: 6A TOGGLE, switch:320-938
- added TP10, TP11, TP12, TP13, TP14, TP15, TP16, TP17, TP18, TP19, TP20, TP21, TP22, TP23, TP24, TP25, TP9: TP_1MM_TH", TP_1MM_TH:TP_1MM_TH"
- BAT1: value (none) -> +9V_BATTERY; OC_FARNELL (none) -> unknown
- C1, C10, C11, C3, C4, C8, C9, J3, J4, J5, J6, J7, J8, J9, LED1, R1, R12, R13, R14, TP1, TP2, TP3, TP4, TP5, TP6, TP7, TP8, U3: OC_FARNELL (none) -> unknown
- C2, C7: value 2.2uF -> 1uF; OC_FARNELL (none) -> unknown
- C5, C6: value 1uF -> 2.2uF; OC_FARNELL (none) -> unknown
- J1, J2: value (none) -> BANANA SOCKET; OC_FARNELL (none) -> unknown
- Q1: value N-HEXFET-2D_SOT232- -> IRF540; device transistor-power:N-HEXFET-2D_SOT232- -> transistor-power:IRF540; MF (none) -> MULTICOMP; MPN (none) -> SR16150; OC_FARNELL (none) -> 1625239
- R10: value 100k -> 1Meg; OC_FARNELL (none) -> unknown
- R11: value 1Meg -> 100R; OC_FARNELL (none) -> unknown
- R2: value 1R -> 1k; OC_FARNELL (none) -> unknown
- R3: value 5R -> 1R; OC_FARNELL (none) -> unknown
- R4: value 10R -> 5k; OC_FARNELL (none) -> unknown
- R5: value 50R -> 5R; OC_FARNELL (none) -> unknown
- R6: value 100R -> 10k; OC_FARNELL (none) -> unknown
- R7: value 1k -> 10R; MF (none) -> COILCRAFT; MPN (none) -> 1008LS-393XJLB; OC_FARNELL (none) -> 2286860
- R8: value 5k -> 100k; OC_FARNELL (none) -> unknown
- R9: value 10k -> 50R; OC_FARNELL (none) -> unknown
- U1: value MAX6225ACSA+ -> MAX6126AASA25+; device MAX6225ACSA+:MAX6225ACSA+ -> MAX6126AASA50+:MAX6126AASA50+; OC_FARNELL (none) -> unknown
- U2: value MAX6250ACSA+ -> MAX6126AASA25+; device MAX62250ACSA+:MAX6250ACSA+ -> MAX6126AASA50+:MAX6126AASA50+; OC_FARNELL (none) -> unknown
Connections:
- removed net +2.5V_OUT: C7.1, J9.1, JP1.1, TP5.1, U1.OUT
- removed net +5.0V_OUT: C8.1, J7.1, JP2.1, TP3.1, U2.OUT
- removed net 18V_PWR: BAT2.V+, J4.1, S1.P
- removed net 9V_PWR: BAT1.V+, BAT2.V-, J8.1
- removed net N$1: TM2.S, U2.TRIM
- removed net N$11: R2.2
- removed net N$25: J6.1, Q1.D, TP2.1
- removed net N$26: C9.1, Q1.G, U3.OUTF
- removed net N$27: C10.1, J2.1, Q1.S, R14.2, TP6.1, U3.OUTS
- removed net N$3: TM1.S, U1.TRIM
- removed net N$7: C4.1, U2.NR
- removed net V_IN: C11.1, C3.1, J5.1, TP1.1, U3.IN
- new net +2.5V_REF: C8.1, J7.1, TP9.1, U2.OUTF, U2.OUTS
- new net +5.0V_REF: C11.1, J9.1, TP11.1, U3.OUTF, U3.OUTS
- new net +6V_IN: F1.1, J1.1
- new net N$15: C7.1, U2.NR
- new net N$22: TP3.1, TP4.1
- new net N$6: C10.1, U3.NR
- new net OUTF: C3.1, Q1.G, U1.OUTF
- new net OUTS: C4.1, J5.1, Q1.S, R14.2, TP6.1, U1.OUTS
- new net Q1_DRAIN: J4.1, Q1.D, TP2.1
- new net VIN_1: F1.2, F2.2, S31.P, S3B.P
- new net V_IN2: C1.1, C5.1, C6.1, C9.1, D1.C, J3.1, R13.2, TP1.1, U1.IN, U2.IN, U3.IN
- net GND: now also J2.1, J6.1, J8.1, KK2.K@1, KK2.K@2, PAD1.P, PAD2.P, PAD3.P, PAD4.P, PAD5.P, PAD6.P, TP10.1, U1.GNDS, U2.GNDS; no longer J1.1, J10.1, J11.1, J3.1, JP1.2, JP2.2, TM1.A, TM2.A, TP4.1, TP8.1
- net N$10: now also R3.1, TP8.1; no longer R2.1
- net N$12: now also R11.2, R2.1, TP15.1, TP24.1; no longer R6.2, R7.1
- net N$13: now also R2.2, R4.1, TP16.1; no longer R7.2, R8.1
- net N$16: now also R4.2, R6.1, TP17.1; no longer R8.2, R9.1
- net N$17: now also R10.1, R8.2, TP19.1; no longer R10.2, R11.1
- net N$18: now also R5.2, R7.1, TP12.1, TP13.1; no longer R3.2, R4.1
- net N$2: now also D1.A1, D1.A2, S31.S, S3B.S; no longer C6.1, U1.NR
- net N$21: now also R10.2, TP20.1; no longer R11.2
- net N$24: now also TP21.1
- net N$28: now also C2.1, U1.NR; no longer C5.1, U3.NR
- net N$29: now also R7.2, R9.1, TP14.1; no longer R4.2, R5.1
- net N$31: now also R3.2, R5.1, TP23.1; no longer R3.1
- net N$34: now also R6.2, R8.1, TP18.1, TP25.1; no longer R10.1, R9.2
- net N$5: now also TP5.1
- net N$8: now also R11.1, R9.2, TP22.1; no longer R5.2, R6.1
- net N$9: now also BAT1.V+, F2.1; no longer C1.1, C2.1, R13.2, S1.S, TM1.E, TM2.E, U1.IN, U2.IN
Other:
- note added: "<- CURRENT METER"
- note added: "MAX6126 needs to be a 4.0v or less due to max rating in the OUTF line"
- note added: "USE THE 9V BATTERY FOR LOW CURRENT REFERENCES. USE THE EXTERNAL PSU FOR HIGH CURRENT REFERENCES."
- note added: "WATTAGE"
- note removed: "8 to 10V = 10pm/V , 10-36V = 2ppm/V"
- note removed: "CHANGE TO SMD VERSION"
- note removed: "CHECK V AND I RATING"
- note removed: "JS202011SCQN"
- note removed: "MAX6126 may need to be a 4.0 or less voltage part due to max rating in the OUTF line"
- note removed: "V_IN = 8 ~ 36V, 10 ~ 36V preferred"
- note removed: "slide switch JS202011SCQN"
- moved on the sheet: BAT1, C1, C10, C11, C2, C3, C4, C5, C6, C7, C8, C9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

Commit message: Added capacitors and inductors
Added capacitors and inductors and corrected some ERC errors
Parts:
- added C12: 10pF, rcl:C-EUC0805
- added C13: 1nF, rcl:C-EUC0805
- added C14: 10nF, rcl:C-EUC0805
- added C15: 100nF, rcl:C-EUC0805
- added C16: 1uF, rcl:C-EUC0805
- added C17: 100uF, rcl:C-EUC0805
- added C18: (no value), rcl:CPOL-USE5-10.5
- added L10: 330nH, rcl:L-USL2825P
- added L5: 10mH, rcl:L-US6000-XXX-RC
- added L7: 1uH, rcl:L-USL1812
- added L8: 100uH, rcl:L-USL1812
- added L9: 1nH, rcl:L-USL1812
- added TP26, TP27, TP28, TP29, TP30, TP31, TP32, TP33, TP34, TP35, TP36, TP37, TP38, TP39, TP41, TP42, TP43, TP44, TP45, TP46, TP47, TP48, TP49, TP51: TP_1MM_TH", TP_1MM_TH:TP_1MM_TH"
- D1: value (none) -> 30A_MIN
- J1, J2: value BANANA SOCKET -> BANANA_CONN
- J3, J4, J5, J6, J7, J8, J9: value (none) -> BANANA_CONN
- LED1: value (none) -> GREEN_LED
- PAD1, PAD2, PAD3, PAD4, PAD5, PAD6: value (none) -> MOUNT_HOLE
- U1, U2: MF (none) -> MAXIM INTEGRATED PRODUCTS; MPN (none) -> MAX6126AASA25+; OC_FARNELL unknown -> 1673170
Connections:
- new net N$1: C12.1, TP26.1
- new net N$11: C17.2, TP30.1
- new net N$14: L7.2, TP37.1
- new net N$19: L8.2, TP38.1
- new net N$20: L5.2, TP39.1
- new net N$23: L9.1, TP42.1
- new net N$25: C18.+, TP41.1
- new net N$26: C18.-, TP51.1
- new net N$3: L9.2, TP35.1
- new net N$48: C12.2, TP27.1
- new net N$49: C13.2, TP32.1
- new net N$50: C14.2, TP33.1
- new net N$51: C15.2, TP29.1
- new net N$52: C16.2, TP31.1
- new net N$53: C13.1, TP34.1
- new net N$54: C14.1, TP44.1
- new net N$55: C15.1, TP46.1
- new net N$56: C16.1, TP47.1
- new net N$57: C17.1, TP48.1
- new net N$59: L5.1, TP43.1
- new net N$60: L8.1, TP49.1
- new net N$61: L7.1, TP45.1
- new net N$62: L10.1, TP28.1
- new net N$7: L10.2, TP36.1
Other:
- note added: "DO NOT CONNECT PINS IC, IC2 TO ANYTHING"
- note added: "REVERSE VOLTAGE PROTECTION"
- note added: "SORT OUT THE CAPS AND INDUCTORS, CHECK THE SEPARATION OF THE TEST POINTS FOR THE TWEEZERS"
- moved on the sheet: F1

Commit message: Updates before PCB release to Fabrication
Updates before PCB release to Fabrication.
Component part numbers for purchase still need specifying.
Parts:
- removed L10: 330nH, rcl:L-USL2825P
- removed L7: 1uH, rcl:L-USL1812
- removed L8: 100uH, rcl:L-USL1812
- removed L9: 1nH, rcl:L-USL1812
- removed R2: 1k, rcl:R-EU_R0805
- removed S3: 6A TOGGLE, switch:320-938
- removed TP51: TP_1MM_TH", TP_1MM_TH:TP_1MM_TH"
- added L1: 1nH, rcl:L-USL1812
- added L2: 330nH, rcl:L-USL2825P
- added L3: 1uH, rcl:L-USL1812
- added L4: 100uH, rcl:L-USL1812
- added R15: 10Meg, rcl:R-EU_R0805
- added S1: 5649A, Switch_320-938_Corrected:320-938
- added TP40: TP_1MM_TH", TP_1MM_TH:TP_1MM_TH"
- C17: value 100uF -> 10uF
- C18: value (none) -> 100uF; OC_FARNELL (none) -> unknown
- C2, C7: value 1uF -> 2.2uF
- C5, C6: value 2.2uF -> 1uF
- D1: value 30A_MIN -> MBR60H100CTG; MF (none) -> ON SEMICONDUCTOR; MPN (none) -> MBR60H100CTG; OC_FARNELL unknown -> 1431072
- L5: OC_FARNELL (none) -> unknown
- R1: value 0.1R -> 2k
- R10: value 1Meg -> 1k
- R11: value 100R -> 5k
- R12: value 10Meg -> 10k
- R13: value 2k -> 100k
- R14: value 5R -> 1Meg
- R3: value 1R -> 5R
- R4: value 5k -> 0.1R
- R5: value 5R -> 1R
- R6: value 10k -> 5R
- R8: value 100k -> 50R
- R9: value 50R -> 100R
- renumbered KK2 to KK1
Connections:
- removed net N$2: D1.A1, D1.A2, S31.S, S3B.S
- removed net N$4: LED1.A, R13.1
- removed net Q1_DRAIN: J4.1, Q1.D, TP2.1
- removed net VIN_1: F1.2, F2.2, S31.P, S3B.P
- removed net V_IN2: C1.1, C5.1, C6.1, C9.1, D1.C, J3.1, R13.2, TP1.1, U1.IN, U2.IN, U3.IN
- new net I_METER-: J6.1, Q1.D, TP4.1
- new net N$30: LED1.A, R1.1
- new net V_IN_1: D1.A1, D1.A2, R1.2, S11.P, S1B.P
- new net V_IN_2: C1.1, C11.1, C2.1, C3.1, D1.C, J5.1, TP3.1, U1.IN, U2.IN, U3.IN
- new net V_IN_A: F1.2, S11.S, S1B.S
- new net V_IN_B: F2.2, S11.O, S1B.O
- net +2.5V_REF: now also J3.1, TP5.1; no longer J7.1, TP9.1
- net +5.0V_REF: now also C9.1, J4.1, TP6.1; no longer C11.1, J9.1, TP11.1
- net GND: now also J9.1, R3.1, TP2.1; no longer J6.1, R14.1, TP10.1
- net N$1: now also TP8.1; no longer TP26.1
- net N$10: now also R4.2, R5.1, TP26.1; no longer R1.2, R3.1, TP8.1
- net N$11: now also TP20.1; no longer TP30.1
- net N$12: now also R10.1, R9.2, TP25.1, TP31.1; no longer R11.2, R2.1, TP15.1, TP24.1
- net N$13: now also R10.2, R11.1, TP34.1; no longer R2.2, R4.1, TP16.1
- net N$14: now also L3.2, TP47.1; no longer L7.2, TP37.1
- net N$15: now also C5.1; no longer C7.1
- net N$16: now also R11.2, R12.1, TP35.1; no longer R4.2, R6.1, TP17.1
- net N$17: now also R13.2, R14.1, TP37.1; no longer R10.1, R8.2, TP19.1
- net N$18: now also R6.2, TP24.1, TP28.1; no longer R5.2, TP12.1, TP13.1
- net N$19: now also L4.2, TP48.1; no longer L8.2, TP38.1
- net N$20: now also TP49.1; no longer TP39.1
- net N$21: now also R14.2, R15.1, TP38.1; no longer R10.2, R12.1, TP20.1
- net N$22: now also TP22.1, TP33.1; no longer TP3.1, TP4.1
- net N$23: now also L1.1, TP40.1; no longer L9.1, TP42.1
- net N$24: now also R15.2, TP39.1; no longer R12.2, TP21.1
- net N$25: now also TP14.1; no longer TP41.1
- net N$26: now also TP21.1; no longer TP51.1
- net N$28: now also C4.1; no longer C2.1
- net N$29: now also R8.1, TP29.1; no longer R9.1, TP14.1
- net N$3: now also L1.2, TP45.1; no longer L9.2, TP35.1
- net N$31: now also R5.2, R6.1, TP27.1; no longer R3.2, R5.1, TP23.1
- net N$34: now also R12.2, R13.1, TP32.1, TP36.1; no longer R6.2, R8.1, TP18.1, TP25.1
- net N$48: now also TP15.1; no longer TP27.1
- net N$49: now also TP16.1; no longer TP32.1
- net N$5: now also R4.1, TP23.1; no longer R1.1, TP5.1
- net N$50: now also TP17.1; no longer TP33.1
- net N$51: now also TP18.1; no longer TP29.1
- net N$52: now also TP19.1; no longer TP31.1
- net N$53: now also TP9.1; no longer TP34.1
- net N$54: now also TP10.1; no longer TP44.1
- net N$55: now also TP11.1; no longer TP46.1
- net N$56: now also TP12.1; no longer TP47.1
- net N$57: now also TP13.1; no longer TP48.1
- net N$59: now also TP44.1; no longer TP43.1
- net N$6: now also C6.1; no longer C10.1
- net N$60: now also L4.1, TP43.1; no longer L8.1, TP49.1
- net N$61: now also L3.1, TP42.1; no longer L7.1, TP45.1
- net N$62: now also L2.1, TP41.1; no longer L10.1, TP28.1
- net N$7: now also L2.2, TP46.1; no longer L10.2, TP36.1
- net N$8: now also R8.2, R9.1, TP30.1; no longer R11.1, R9.2, TP22.1
- net OUTF: now also C7.1; no longer C3.1
- net OUTS: now also C10.1, J7.1, R3.2, TP1.1; no longer C4.1, J5.1, R14.2, TP6.1
Other:
- note added: "<- LOAD"
- note added: "FIX THE CAPS AND INDUCTORS, CHECK THE SEPARATION OF THE TEST POINTS FOR THE TWEEZERS"
- note added: "NO CONNECT PINS IC, IC2"
- note added: "ON/OFF/ON"
- note removed: "DO NOT CONNECT PINS IC, IC2 TO ANYTHING"
- note removed: "SORT OUT THE CAPS AND INDUCTORS, CHECK THE SEPARATION OF THE TEST POINTS FOR THE TWEEZERS"
- note removed: "WATTAGE"
- moved on the sheet: BAT1, C10, C11, C12, C13, C14, C15, C16, C17, C18, C2, C3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
